File: eagle/v1-1-0b.sch (EAGLE design)
At the start: 176 parts, among them J1 CR22A-44D-2.54DSA(70), J3 26-60-4040, J4 AUDIO_JACK_3.5MM_PTH, J5 DIN5, SW1 3PDT-AQ-SWITCH, SW2 9077-1, U10 7805, U11 74LS10N, U13 74LS04N, U14 4528N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

Commit message: Schematic and Board updates
Parts:
- C40, C41, C42: value .02u -> .02uF
Changed lines of the file:
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@@
 <part name="R31" library="aq-rcl" deviceset="R-US_" device="0207/10" package3d_urn="urn:adsk.eagle:package:23491/2" value="3.9k"/>
 <part name="R29" library="aq-rcl" deviceset="R-US_" device="0207/10" package3d_urn="urn:adsk.eagle:package:23491/2" value="100"/>
-<part name="C42" library="aq-rcl" deviceset="C-US" device="050-025X090" value=".02u"/>
+<part name="C42" library="aq-rcl" deviceset="C-US" device="050-025X090" value=".02uF"/>
 <part name="D11" library="aq-diode" deviceset="1N4148" device=""/>
 <part name="D2" library="aq-diode" deviceset="1N4148" device="-12" value="1N4148H"/>
@@
 <part name="L8" library="aq-rcl" deviceset="L-US" device="TFI0305" package3d_urn="urn:adsk.eagle:package:23529/1"/>
 <part name="L6" library="aq-rcl" deviceset="L-US" device="TFI0305" package3d_urn="urn:adsk.eagle:package:23529/1"/>
-<part name="C40" library="aq-rcl" deviceset="C-US" device="050-025X090" value=".02u"/>
-<part name="C41" library="aq-rcl" deviceset="C-US" device="050-025X090" value=".02u"/>
+<part name="C40" library="aq-rcl" deviceset="C-US" device="050-025X090" value=".02uF"/>
+<part name="C41" library="aq-rcl" deviceset="C-US" device="050-025X090" value=".02uF"/>
 <part name="J3" library="26-60-4040" deviceset="26-60-4040" device=""/>
 <part name="C4" library="aq-rcl" deviceset="C-US" device="050-025X090" value=".1uF"/>
