File: eagle/v1-1-0c.sch (EAGLE design)
At the start: 180 parts, among them J1 CR22A-44D-2.54DSA(70), J3 26-60-4040, J4 AUDIO_JACK_3.5MM_PTH, J5 DIN5, SW1 3PDT-AQ-SWITCH, SW2 9077-1, U10 7805, U11 74LS10N, U13 74LS04N, U14 4528N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

Commit message: 09 DEC Update
Parts:
- removed TR1: (no value), aq-rcl:R-TRIMM10MM-DUAL
- added L-V1: 10uH @ 4.43MHz, aq-rcl:L-VAR-IND
- C32: value 100pF -> 100pF/47pF
Connections:
- net GND: no longer TR1.S
- net N$691: now also L-V1.P$1; no longer TR1.E
- net VPP: now also L-V1.P$2; no longer TR1.A
Other:
- note added: "09 DEC 2020"
- note added: "Optional Chroma Band Limiter"
- note removed: "06 NOV 2020"
- moved on the sheet: C32
Changed lines of the file:
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@@
 <part name="C34" library="aq-rcl" deviceset="C-US" device="025-024X044" package3d_urn="urn:adsk.eagle:package:23630/1" value="2pF/∞"/>
 <part name="C35" library="aq-rcl" deviceset="C-US" device="050-025X090" value=".1uF/∞"/>
-<part name="C32" library="aq-rcl" deviceset="C-US" device="025-024X044" package3d_urn="urn:adsk.eagle:package:23630/1" value="100pF"/>
+<part name="C32" library="aq-rcl" deviceset="C-US" device="025-024X044" package3d_urn="urn:adsk.eagle:package:23630/1" value="100pF/47pF"/>
 <part name="C14" library="aq-rcl" deviceset="C-US" device="050-024X044" package3d_urn="urn:adsk.eagle:package:23643/1" value=".022uF"/>
 <part name="C39" library="aq-rcl" deviceset="C-US" device="050-024X044" package3d_urn="urn:adsk.eagle:package:23643/1" value="56pF/∞"/>
@@
 <part name="GND25" library="supply1" library_urn="urn:adsk.eagle:library:371" deviceset="GND" device=""/>
 <part name="J4" library="SparkFun-Connectors" library_urn="urn:adsk.eagle:library:513" deviceset="AUDIO_JACK_3.5MM" device="_PTH" package3d_urn="urn:adsk.eagle:package:37997/1"/>
-<part name="TR1" library="aq-rcl" deviceset="R-TRIMM" device="10MM-DUAL"/>
-<part name="GND31" library="supply1" library_urn="urn:adsk.eagle:library:371" deviceset="GND" device=""/>
 <part name="P+22" library="supply1" library_urn="urn:adsk.eagle:library:371" deviceset="VCC" device=""/>
 <part name="GND33" library="supply1" library_urn="urn:adsk.eagle:library:371" deviceset="GND" device=""/>
 <part name="SUPPLY2" library="supply2" library_urn="urn:adsk.eagle:library:372" deviceset="VEE" device=""/>
 <part name="P+23" library="supply1" library_urn="urn:adsk.eagle:library:371" deviceset="VCC" device=""/>
-<part name="SUPPLY5" library="supply2" library_urn="urn:adsk.eagle:library:372" deviceset="VPP" device=""/>
 <part name="GND35" library="supply1" library_urn="urn:adsk.eagle:library:371" deviceset="GND" device=""/>
 <part name="C38" library="aq-rcl" deviceset="C-US" device="050-025X085" value="100pF"/>
@@
 <part name="GND36" library="supply1" library_urn="urn:adsk.eagle:library:371" deviceset="GND" device=""/>
 <part name="C44" library="aq-rcl" deviceset="C-US" device="050-024X044" package3d_urn="urn:adsk.eagle:package:23643/1" value="∞/22pF"/>
+<part name="L-V1" library="aq-rcl" deviceset="L-VAR-IND" device="" value="10uH @ 4.43MHz"/>
 </parts>
 <sheets>
@@
 <wire x1="261.62" y1="15.24" x2="261.62" y2="5.08" width="0.1524" layer="97"/>
 <wire x1="261.62" y1="5.08" x2="347.98" y2="5.08" width="0.1524" layer="97"/>
-<text x="304.8" y="7.62" size="5.08" layer="97" align="bottom-center">06 NOV 2020</text>
+<text x="304.8" y="7.62" size="5.08" layer="97" align="bottom-center">09 DEC 2020</text>
 <wire x1="347.98" y1="15.24" x2="347.98" y2="25.4" width="0.1524" layer="97"/>
 <wire x1="347.98" y1="25.4" x2="261.62" y2="25.4" width="0.1524" layer="97"/>
@@
 <text x="401.32" y="165.1" size="1.016" layer="97" distance="25" rot="R180" align="center">NTSC Close
 for 2Φ</text>
+<wire x1="581.152" y1="251.46" x2="598.424" y2="251.46" width="0.1524" layer="97" style="shortdash"/>
+<wire x1="598.424" y1="251.46" x2="598.424" y2="273.05" width="0.1524" layer="97" style="shortdash"/>
+<wire x1="598.424" y1="273.05" x2="581.152" y2="273.05" width="0.1524" layer="97" style="shortdash"/>
+<wire x1="581.152" y1="273.05" x2="581.152" y2="251.46" width="0.1524" layer="97" style="shortdash"/>
+<text x="589.788" y="248.92" size="1.524" layer="97" align="center">Optional
+Chroma Band Limiter</text>
 </plain>
 <instances>
@@
 <attribute name="VALUE" x="514.858" y="130.175" size="1.778" layer="96"/>
 </instance>
-<instance part="C32" gate="G$1" x="589.28" y="266.7" smashed="yes" rot="MR90">
-<attribute name="NAME" x="587.502" y="269.875" size="1.778" layer="95" rot="MR0"/>
-<attribute name="VALUE" x="590.169" y="266.954" size="1.778" layer="96" rot="MR90"/>
+<instance part="C32" gate="G$1" x="590.55" y="266.7" smashed="yes" rot="MR90">
+<attribute name="NAME" x="595.884" y="268.097" size="1.778" layer="95" rot="MR0"/>
+<attribute name="VALUE" x="585.724" y="263.525" size="1.27" layer="96" rot="MR180"/>
 </instance>
 <instance part="C14" gate="G$1" x="574.04" y="266.7" smashed="yes" rot="MR270">
@@
 <attribute name="NAME" x="190.5" y="139.192" size="1.778" layer="95" font="vector" rot="MR180"/>
 </instance>
-<instance part="TR1" gate="G$1" x="589.28" y="256.54" smashed="yes" rot="MR270">
-<attribute name="NAME" x="592.328" y="260.223" size="1.778" layer="95" rot="MR0"/>
-<attribute name="VALUE" x="593.09" y="260.35" size="1.778" layer="96" rot="MR0"/>
-</instance>
-<instance part="GND31" gate="1" x="589.28" y="246.38" smashed="yes" rot="MR0">
-<attribute name="VALUE" x="591.82" y="243.84" size="1.778" layer="96" rot="MR0"/>
-</instance>
 <instance part="P+22" gate="VCC" x="261.62" y="154.94" smashed="yes" rot="R270">
 <attribute name="VALUE" x="262.382" y="154.94" size="1.778" layer="96"/>
@@
 <attribute name="VALUE" x="370.84" y="86.36" size="1.778" layer="96" rot="R90"/>
 </instance>
-<instance part="SUPPLY5" gate="G$1" x="596.9" y="269.24" smashed="yes" rot="MR0">
-<attribute name="VALUE" x="598.805" y="272.415" size="1.778" layer="96" rot="MR0"/>
-</instance>
 <instance part="GND35" gate="1" x="447.04" y="134.62" smashed="yes" rot="R270">
 <attribute name="VALUE" x="444.5" y="137.16" size="1.778" layer="96" rot="R270"/>
@@
 <attribute name="VALUE" x="598.678" y="72.517" size="1.778" layer="96" rot="R180"/>
 </instance>
+<instance part="L-V1" gate="G$1" x="589.28" y="256.54" smashed="yes" rot="R270">
+<attribute name="VALUE" x="589.28" y="254" size="1.27" layer="96" align="center"/>
+<attribute name="NAME" x="590.55" y="259.842" size="1.778" layer="95" align="center"/>
+</instance>
 </instances>
 <busses>
@@
 </segment>
 <segment>
-<pinref part="TR1" gate="G$1" pin="S"/>
-<wire x1="589.28" y1="251.46" x2="589.28" y2="248.92" width="0.1524" layer="91"/>
-<pinref part="GND31" gate="1" pin="GND"/>
-</segment>
-<segment>
 <pinref part="C43" gate="G$1" pin="2"/>
 <wire x1="604.52" y1="81.28" x2="599.44" y2="81.28" width="0.1524" layer="91"/>
@@
 <wire x1="566.42" y1="330.2" x2="566.42" y2="335.28" width="0.1524" layer="91"/>
 <junction x="566.42" y="335.28"/>
+<pinref part="C32" gate="G$1" pin="1"/>
+<wire x1="593.09" y1="266.7" x2="596.9" y2="266.7" width="0.1524" layer="91"/>
+<wire x1="596.9" y1="256.54" x2="594.36" y2="256.54" width="0.1524" layer="91"/>
+<wire x1="596.9" y1="266.7" x2="596.9" y2="256.54" width="0.1524" layer="91"/>
+<pinref part="L-V1" gate="G$1" pin="P$2"/>
+<wire x1="596.9" y1="266.7" x2="596.9" y2="271.78" width="0.1524" layer="91"/>
+<junction x="596.9" y="266.7"/>
+<wire x1="596.9" y1="271.78" x2="571.5" y2="271.78" width="0.1524" layer="91"/>
+<wire x1="571.5" y1="271.78" x2="571.5" y2="274.32" width="0.1524" layer="91"/>
+<wire x1="571.5" y1="274.32" x2="566.42" y2="274.32" width="0.1524" layer="91"/>
+<junction x="566.42" y="274.32"/>
 </segment>
 <segment>
@@
 </segment>
 <segment>
-<pinref part="C32" gate="G$1" pin="1"/>
-<wire x1="591.82" y1="266.7" x2="596.9" y2="266.7" width="0.1524" layer="91"/>
-<pinref part="TR1" gate="G$1" pin="A"/>
-<wire x1="596.9" y1="256.54" x2="594.36" y2="256.54" width="0.1524" layer="91"/>
-<wire x1="596.9" y1="266.7" x2="596.9" y2="256.54" width="0.1524" layer="91"/>
-<pinref part="SUPPLY5" gate="G$1" pin="VPP"/>
-<junction x="596.9" y="266.7"/>
-</segment>
-<segment>
 <pinref part="JP4" gate="A" pin="2"/>
 <pinref part="SUPPLY7" gate="G$1" pin="VPP"/>
@@
 <pinref part="C14" gate="G$1" pin="2"/>
 <pinref part="C32" gate="G$1" pin="2"/>
-<wire x1="584.2" y1="266.7" x2="581.66" y2="266.7" width="0.1524" layer="91"/>
-<pinref part="TR1" gate="G$1" pin="E"/>
-<wire x1="584.2" y1="256.54" x2="581.66" y2="256.54" width="0.1524" layer="91"/>
-<wire x1="581.66" y1="266.7" x2="581.66" y2="256.54" width="0.1524" layer="91"/>
-<wire x1="579.12" y1="266.7" x2="581.66" y2="266.7" width="0.1524" layer="91"/>
-<junction x="581.66" y="266.7"/>
+<wire x1="585.47" y1="266.7" x2="582.676" y2="266.7" width="0.1524" layer="91"/>
+<wire x1="584.2" y1="256.54" x2="582.676" y2="256.54" width="0.1524" layer="91"/>
+<wire x1="582.676" y1="266.7" x2="582.676" y2="256.54" width="0.1524" layer="91"/>
+<wire x1="579.12" y1="266.7" x2="582.676" y2="266.7" width="0.1524" layer="91"/>
+<junction x="582.676" y="266.7"/>
+<pinref part="L-V1" gate="G$1" pin="P$1"/>
 </segment>
 </net>

Commit message: January fixes
Other:
- note added: "15 JAN 2021"
- note added: "NTSC to JP3 TEA1002 PALSW"
- note added: "PAL to JP3 TEA1002 PALSW"
- note removed: "09 DEC 2020"
- note removed: "NTSC to JP4 TEA1002 PALSW"
- note removed: "PAL to JP4 TEA1002 PALSW"
Changed lines of the file:
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@@
 <wire x1="261.62" y1="15.24" x2="261.62" y2="5.08" width="0.1524" layer="97"/>
 <wire x1="261.62" y1="5.08" x2="347.98" y2="5.08" width="0.1524" layer="97"/>
-<text x="304.8" y="7.62" size="5.08" layer="97" align="bottom-center">09 DEC 2020</text>
+<text x="304.8" y="7.62" size="5.08" layer="97" align="bottom-center">15 JAN 2021</text>
 <wire x1="347.98" y1="15.24" x2="347.98" y2="25.4" width="0.1524" layer="97"/>
 <wire x1="347.98" y1="25.4" x2="261.62" y2="25.4" width="0.1524" layer="97"/>
@@
 <wire x1="59.436" y1="59.436" x2="59.436" y2="67.818" width="0.1524" layer="97" style="shortdash"/>
 <text x="343.154" y="187.96" size="1.27" layer="97" distance="25" align="center">(NTSC to GND)</text>
-<text x="344.424" y="195.072" size="1.016" layer="97" distance="25" rot="R180" align="center">NTSC to JP4
+<text x="344.424" y="195.072" size="1.016" layer="97" distance="25" rot="R180" align="center">NTSC to JP3
 TEA1002 PALSW</text>
-<text x="268.732" y="258.064" size="1.016" layer="97" distance="25" rot="R180" align="center">PAL to JP4
+<text x="268.732" y="258.064" size="1.016" layer="97" distance="25" rot="R180" align="center">PAL to JP3
 TEA1002 PALSW</text>
 <wire x1="467.36" y1="109.22" x2="467.36" y2="95.504" width="0.254" layer="97"/>

Commit message: Rev C Full Release
Parts:
- C16: value 82pF/∞ -> ∞/82pF
Other:
- note added: "19 JAN 2021"
- note removed: "15 JAN 2021"
Changed lines of the file:
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@@
 <part name="C19" library="aq-rcl" deviceset="C-US" device="050-024X044" package3d_urn="urn:adsk.eagle:package:23643/1" value="82pF"/>
 <part name="C18" library="aq-rcl" deviceset="C-US" device="050-024X044" package3d_urn="urn:adsk.eagle:package:23643/1" value="82pF"/>
-<part name="C16" library="aq-rcl" deviceset="C-US" device="050-024X044" package3d_urn="urn:adsk.eagle:package:23643/1" value="82pF/∞"/>
+<part name="C16" library="aq-rcl" deviceset="C-US" device="050-024X044" package3d_urn="urn:adsk.eagle:package:23643/1" value="∞/82pF"/>
 <part name="L5" library="aq-rcl" deviceset="L-US" device="TFI0305" package3d_urn="urn:adsk.eagle:package:23529/1"/>
 <part name="L7" library="aq-rcl" deviceset="L-US" device="TFI0305" package3d_urn="urn:adsk.eagle:package:23529/1"/>
@@
 <wire x1="261.62" y1="15.24" x2="261.62" y2="5.08" width="0.1524" layer="97"/>
 <wire x1="261.62" y1="5.08" x2="347.98" y2="5.08" width="0.1524" layer="97"/>
-<text x="304.8" y="7.62" size="5.08" layer="97" align="bottom-center">15 JAN 2021</text>
+<text x="304.8" y="7.62" size="5.08" layer="97" align="bottom-center">19 JAN 2021</text>
 <wire x1="347.98" y1="15.24" x2="347.98" y2="25.4" width="0.1524" layer="97"/>
 <wire x1="347.98" y1="25.4" x2="261.62" y2="25.4" width="0.1524" layer="97"/>
