File: eagle/v1-1-0x.brd (EAGLE design)
At the start: 313 x 132.9 mm, 182 parts, among them J1 CR22A-44D-2.54DSA(70), J3 26-60-4040, J4 AUDIO_JACK_3.5MM_PTH, J5 DIN5, SW1 3PDT-AQ-SWITCH, SW2 9077-1, U10 7805, U11 74LS10N, U13 74LS04N, U14 4528N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

Commit message: Rev D updates
Parts:
- removed U$1: (no value), aquarius:AQUARIUS-LOGO-SMALL
- added IC2, SYSROM-ALT: 27C512AP, microchip:DIL28-6
- JP7: device aquarius2:1X02 -> aquarius2:2X03
- moved JP7 165.0 mm to (-4.06, -31.8), turned to 0 degrees
Connections:
- new net N$112: JP7.1
- new net N$116: JP7.3
- new net N$117: JP7.5
- new net N$119: JP7.2
- new net N$120: JP7.4
- new net N$124: JP7.6
- net !ROM: now also SYSROM-ALT.20, SYSROM-ALT.22
- net A00: now also SYSROM-ALT.10
- net A01: now also SYSROM-ALT.9
- net A02: now also SYSROM-ALT.8
- net A03: now also SYSROM-ALT.7
- net A04: now also SYSROM-ALT.6
- net A05: now also SYSROM-ALT.5
- net A06: now also SYSROM-ALT.4
- net A07: now also SYSROM-ALT.3
- net A08: now also SYSROM-ALT.25
- net A09: now also SYSROM-ALT.24
- net A10: now also SYSROM-ALT.21
- net A11: now also SYSROM-ALT.23
- net A12: now also SYSROM-ALT.2
- net D00: now also SYSROM-ALT.11
- net D01: now also SYSROM-ALT.12
- net D02: now also SYSROM-ALT.13
- net D03: now also SYSROM-ALT.15
- net D04: now also SYSROM-ALT.16
- net D05: now also SYSROM-ALT.17
- net D06: now also SYSROM-ALT.18
- net D07: now also SYSROM-ALT.19
- net GND: now also IC2.14, SYSROM-ALT.14; no longer JP7.2
- net VCC: now also IC2.28, SYSROM-ALT.28; no longer JP7.1
Routing:
- net GND: track 653.8 -> 636.6 mm
- net VCC: track 1100.0 -> 1088.3 mm
- net A12: track 258.5 -> 268.5 mm
- net A11: track 258.7 -> 264.8 mm
- net D06: track 202.3 -> 207.9 mm, vias 3 -> 2
- net N$40: track 0.00 -> 5.59 mm
- net N$38: track 0.00 -> 4.63 mm
- net A08: track 224.4 -> 228.9 mm
- net N$46: track 0.00 -> 4.42 mm
- net N$47: track 0.00 -> 4.42 mm
- net N$13: track 0.00 -> 4.37 mm
- net N$48: track 0.00 -> 4.27 mm
- net N$39: track 0.00 -> 4.27 mm
- net N$41: track 0.00 -> 3.62 mm
- net N$44: track 0.00 -> 3.36 mm
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- added copper zone on layer 16, net LOGO
- added copper zone on layer 16, net N$1120
- added copper zone on layer 16, net N$1313
- added copper zone on layer 16, net N$1381
- added copper zone on layer 16, net N$1382
- added copper zone on layer 16, net N$1386
- added copper zone on layer 16, net N$1393
- added copper zone on layer 16, net N$966
- removed copper zone on layer 16, net N$31
- removed copper zone on layer 16, net N$37
- removed copper zone on layer 16, net N$620
Other:
- board text added: "Aquarius Motherboard v1.1.0 Rev C - 31 JAN 2022 by Sean Harrington, sph@1stage.com"
- board text removed: "+5v"
- board text removed: "Motherboard v1.1.0 Rev D - 30 APR 2022 by Sean Harrington, sph@1stage.com"
