File: eagle/v1-1-0x.sch (EAGLE design)
At the start: 181 parts, among them J1 CR22A-44D-2.54DSA(70), J3 26-60-4040, J4 AUDIO_JACK_3.5MM_PTH, J5 DIN5, SW1 3PDT-AQ-SWITCH, SW2 9077-1, U10 7805, U11 74LS10N, U13 74LS04N, U14 4528N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

Commit message: Rev D updates
Parts:
- added IC2, SYSROM-ALT: 27C512AP, microchip:27C512AP
- JP7: device aquarius2:PINHD-1X2 -> aquarius2:PINHD-2X3
Connections:
- new net N$112: JP7.1
- new net N$116: JP7.3
- new net N$117: JP7.5
- new net N$119: JP7.2
- new net N$120: JP7.4
- new net N$124: JP7.6
- net !ROM: now also SYSROM-ALT.!CE, SYSROM-ALT.VPP/!OE
- net A00: now also SYSROM-ALT.A0
- net A01: now also SYSROM-ALT.A1
- net A02: now also SYSROM-ALT.A2
- net A03: now also SYSROM-ALT.A3
- net A04: now also SYSROM-ALT.A4
- net A05: now also SYSROM-ALT.A5
- net A06: now also SYSROM-ALT.A6
- net A07: now also SYSROM-ALT.A7
- net A08: now also SYSROM-ALT.A8
- net A09: now also SYSROM-ALT.A9
- net A10: now also SYSROM-ALT.A10
- net A11: now also SYSROM-ALT.A11
- net A12: now also SYSROM-ALT.A12
- net D00: now also SYSROM-ALT.D0
- net D01: now also SYSROM-ALT.D1
- net D02: now also SYSROM-ALT.D2
- net D03: now also SYSROM-ALT.D3
- net D04: now also SYSROM-ALT.D4
- net D05: now also SYSROM-ALT.D5
- net D06: now also SYSROM-ALT.D6
- net D07: now also SYSROM-ALT.D7
- net GND: now also SYSROM-ALT.GND; no longer JP7.2
- net VCC: now also SYSROM-ALT.VCC; no longer JP7.1
Other:
- note added: "31 JAN 2022"
- note added: "AUX Power Header"
- note added: "Aquarius Motherboard v1-1-0 - Rev C"
- note removed: "30 APR 2022"
- note removed: "AUX Power Headers"
- note removed: "Aquarius Motherboard v1-1-0 - Rev D"
